File: copilot-ext-3xUSB.kicad_sch (KiCad schematic)
At the start: 45 parts, among them J1 Conn_01x06_Socket, J10 Conn_01x03_Socket, J11 Conn_01x03_Socket, J2 Conn_01x06_Socket, J3 USB_C_Receptacle_USB2.0, J4 USB_C_Receptacle_USB2.0, J5 USB_C_Receptacle_USB2.0, J6 USB_A, J7 USB_A, J8 USB_A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

Commit message: Improvements and fixes
- Change configuration pins
- Add documentaiton on back of the board
- increase type-C power line width
- Align headers

Signed-off-by: Stoyan Bogdanov <sbogdanov@baylibre.com>
Parts:
- removed J10, J11, J9: Conn_01x03_Socket, Connector_PinHeader_2.54mm:PinHeader_1x03_P2.54mm_Vertical, symbol Connector:Conn_01x03_Socket
- added J10, J11, J9: Conn_02x03_Odd_Even, Connector_PinHeader_2.54mm:PinHeader_2x03_P2.54mm_Vertical, symbol Connector_Generic:Conn_02x03_Odd_Even
- J1: footprint Connector_PinSocket_2.54mm:PinSocket_1x06_P2.54mm_Vertical_SMD_Pin1Right -> Connector_PinHeader_2.54mm:PinHeader_1x06_P2.54mm_Vertical_SMD_Pin1Right
- J2: footprint Connector_PinHeader_2.54mm:PinHeader_1x06_P2.54mm_Vertical_SMD_Pin1Right -> Connector_PinSocket_2.54mm:PinSocket_1x06_P2.54mm_Vertical_SMD_Pin1Right
Connections:
- net GPIO_1: now also J10.5 (Pin_5), J11.5 (Pin_5), J9.5 (Pin_5)
- net GPIO_2: now also J10.3 (Pin_3), J11.3 (Pin_3), J9.3 (Pin_3)
- net GPIO_3: now also J10.1 (Pin_1), J11.1 (Pin_1), J9.1 (Pin_1)
- net GPIO_JP_1: now also J9.2 (Pin_2), J9.4 (Pin_4), J9.6 (Pin_6)
- net GPIO_JP_2: now also J10.2 (Pin_2), J10.4 (Pin_4), J10.6 (Pin_6)
- net GPIO_JP_3: now also J11.2 (Pin_2), J11.4 (Pin_4), J11.6 (Pin_6)
- no-connect marks 0 -> 12
Other:
- moved on the sheet: C1, C2, C3, C4, C5, C6, H1, H2, H3, H4, J1, J2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

Commit message: Export locally and relink project:
- Export 3D models
- Export Schematic symbols
- Export PCB footprints
- Relink local 3D models to local footprints
- Relink local schematic symbols to local footprints

Signed-off-by: Stoyan Bogdanov <sbogdanov@baylibre.com>
Parts:
- C1, C2, C3, C4, C5, C6: footprint Capacitor_SMD:C_0805_2012Metric -> usb2-extension:C_0805_2012Metric; symbol Library:C -> usb2-extension:C
- D1, D2, D3: footprint LED_SMD:LED_0805_2012Metric -> usb2-extension:LED_0805_2012Metric; symbol Library:LED -> usb2-extension:LED
- H1, H2, H3, H4: footprint MountingHole:MountingHole_2.7mm -> usb2-extension:MountingHole_2.7mm; symbol Library:MountingHole -> usb2-extension:MountingHole
- J1: footprint Connector_PinHeader_2.54mm:PinHeader_1x06_P2.54mm_Vertical_SMD_Pin1Right -> usb2-extension:PinHeader_1x06_P2.54mm_Vertical_SMD_Pin1Right; symbol Library:Conn_01x06_Socket -> usb2-extension:Conn_01x06_Socket
- J10, J11, J9: footprint Connector_PinHeader_2.54mm:PinHeader_2x03_P2.54mm_Vertical -> usb2-extension:PinHeader_2x03_P2.54mm_Vertical; symbol Connector_Generic:Conn_02x03_Odd_Even -> usb2-extension:Conn_02x03_Odd_Even
- J2: footprint Connector_PinSocket_2.54mm:PinSocket_1x06_P2.54mm_Vertical_SMD_Pin1Right -> usb2-extension:PinSocket_1x06_P2.54mm_Vertical_SMD_Pin1Right; symbol Library:Conn_01x06_Socket -> usb2-extension:Conn_01x06_Socket
- J3, J4, J5: footprint Connector_USB:USB_C_Receptacle_GCT_USB4085 -> usb2-extension:USB_C_Receptacle_GCT_USB4085; symbol Library:USB_C_Receptacle_USB2.0 -> usb2-extension:USB_C_Receptacle_USB2.0
- J6, J7, J8: footprint Connector_USB:USB_A_Wuerth_614004134726_Horizontal -> usb2-extension:USB_A_Wuerth_614004134726_Horizontal; symbol Library:USB_A -> usb2-extension:USB_A
- Q1, Q2, Q3: footprint Package_SO:SO-8_3.9x4.9mm_P1.27mm -> usb2-extension:SO-8_3.9x4.9mm_P1.27mm; symbol Library:BUK7M27-80EX_1 -> usb2-extension:BUK7M27-80EX_1
- Q4, Q5, Q6: footprint Package_TO_SOT_SMD:SOT-23 -> usb2-extension:SOT-23; symbol Library:BSS138 -> usb2-extension:BSS138
- R1, R2, R3, R4, R5, R6: footprint Resistor_SMD:R_0805_2012Metric -> usb2-extension:R_0805_2012Metric; symbol Library:R -> usb2-extension:R
- R10, R11, R12: footprint Resistor_SMD:R_1206_3216Metric -> usb2-extension:R_1206_3216Metric; symbol Library:R -> usb2-extension:R
- R7, R8, R9: footprint Resistor_SMD:R_0603_1608Metric -> usb2-extension:R_0603_1608Metric; symbol Library:R -> usb2-extension:R
- U1, U2, U3: footprint Package_TO_SOT_SMD:SOT-23-8 -> usb2-extension:SOT-23-8; symbol Library:LM74502 -> usb2-extension:LM74502
