File: copilot-ext-3xUSB.kicad_sch (KiCad schematic)
At the start: 45 parts, among them J1 Conn_01x06_Socket, J10 Conn_02x03_Odd_Even, J11 Conn_02x03_Odd_Even, J2 Conn_01x06_Socket, J3 USB_C_Receptacle_USB2.0, J4 USB_C_Receptacle_USB2.0, J5 USB_C_Receptacle_USB2.0, J6 USB_A, J7 USB_A, J8 USB_A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

Commit message: Assign a manufacturer part number to each board component.
Signed-off-by: Adrien Ricciardi <aricciardi@baylibre.com>
Parts:
- C1, C2, C3: AISLER_MPN 100n 100V X7R 0805 -> (none); MPN (none) -> 100n 35V X7R 0805; Value2 100V -> 35V
- C4, C5, C6: AISLER_MPN 220n 35V X7R 0805 -> (none); MPN (none) -> 220n 35V X7R 0805
- D1, D2, D3: AISLER_MPN 150080SS75000 -> (none); MPN (none) -> 150080SS75000
- J1: MPN (none) -> 10129380-906001ALF
- J10, J11, J9: MPN (none) -> 10129382-906003BLF
- J2: MPN (none) -> 1241152-6
- J3, J4, J5: MPN (none) -> USB4085-GF-A
- J6, J7, J8: MPN (none) -> 614004134726
- Q1, Q2, Q3: AISLER_MPN DMT6013LSS -> (none); MPN (none) -> DMT6013LSS-13
- Q4, Q5, Q6: AISLER_MPN BSS138P,215 -> (none); MPN (none) -> BSS138P,215
- R1, R3, R5: AISLER_MPN 100K 1% 0805 -> (none); MPN (none) -> 100K 1% 0805
- R10, R11, R12: AISLER_MPN 240 5% 1206 -> (none); MPN (none) -> 240 5% 1206
- R2, R4, R6: AISLER_MPN 2.4K 1% 0805 -> (none); MPN (none) -> 2.4K 1% 0805
- R7, R8, R9: AISLER_MPN 10K 1% 0603 -> (none); MPN (none) -> 10K 1% 0603
- U1, U2, U3: AISLER_MPN LM74502DDFR -> (none); MPN (none) -> LM74502DDFR

Commit message: Add title, revision and company name to the schematic and the PCB sheets.
Signed-off-by: Adrien Ricciardi <aricciardi@baylibre.com>
Other:
- company: (none) -> (C) BayLibre SAS
- title: (none) -> Copilot 3xUSB extension
Changed lines of the file:
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@@
 	(generator_version "9.0")
 	(paper "A2")
+	(title_block
+		(title "Copilot 3xUSB extension")
+		(rev "1.2")
+		(company "(C) BayLibre SAS")
+	)
 	(text "Disable channel power\non boot and when jumper\nis not fitted."
 		(exclude_from_sim no)
